Commit message: urdf v1.0.0 done
Signed-off-by: adrianco <adrian.cobo.mh@gmail.com>

File: description/jetson.xacro (robot description, xacro)
@@ -13,5 +13,5 @@
         <link name="jetson_link">
             <visual name="">
-                <origin xyz="0.0 0.0 0.00" rpy="0.0 0.0 0.0"/>
+                <origin xyz="0.0 0.0 0.0" rpy="0.0 0.0 0.0"/>
                 <geometry>
                     <box size="0.105 0.105 0.073"/>
@@ -20,5 +20,5 @@
             </visual>
             <collision>
-                <origin xyz="0.0 0.0 0.00" rpy="0.0 0.0 0.0"/>
+                <origin xyz="0.0 0.0 0.0" rpy="0.0 0.0 0.0"/>
                 <geometry>
                     <box size="0.105 0.105 0.073"/>

File: description/lidar.xacro (robot description, xacro)
@@ -9,7 +9,7 @@
             <xacro:insert_block name="origin" />
             <parent link="${parent}"/>
-            <child link="lidar_link" />
+            <child link="rs_lidar" />
         </joint>
-        <link name="lidar_link">
+        <link name="rs_lidar">
             <visual name="">
                 <origin xyz="0.0 0.0 0.0" rpy="0.0 0.0 0.0"/>

File: description/soporte.xacro (robot description, xacro)
@@ -5,5 +5,5 @@
     <xacro:arg name="use_mesh" default="true" />
     <xacro:include filename="inertial_macros.xacro"/>
-    <xacro:include filename="soporte_inferior.xacro" />
+    <xacro:include filename="soporte_core.xacro" />
     <xacro:include filename="lidar.xacro" />
     <xacro:include filename="jetson.xacro" />
@@ -12,6 +12,6 @@
         <origin xyz="0.0 0.0 0.0575" rpy="0 0 0"/>
     </xacro:lidar>
-    <xacro:jetson parent="lidar_chassis">
-        <origin xyz="0.0 0.0 -0.064" rpy="0 0 0"/>
+    <xacro:jetson parent="base_footprint">
+        <origin xyz="0.0 0.0 -0.0365" rpy="0 0 0"/>
     </xacro:jetson>
     <xacro:sensor_d435 parent="camera_attachment_link" use_nominal_extrinsics="$(arg use_nominal_extrinsics)" add_plug="$(arg add_plug)" use_mesh="$(arg use_mesh)">

File: description/soporte_core.xacro (robot description, xacro)
@@ -15,5 +15,5 @@
     <link name="base_footprint"></link>
     <joint name="base_chassis_joint" type="fixed">
-        <origin xyz="0.0 0.0 0.0025" rpy="0.0 0.0 0.0"/>
+        <origin xyz="0.0 0.0 0.0" rpy="0.0 0.0 0.0"/>
         <parent link="base_footprint"/>
         <child link="base_chassis"/>
@@ -28,5 +28,5 @@
         </visual>
         <collision>
-            <origin xyz="0 0.0 0.0" rpy="0.0 0.0 0.0"/>
+            <origin xyz="0 0.0 -0.005" rpy="0.0 0.0 0.0"/>
             <geometry>
                 <mesh filename="package://perception_system/meshes/base.dae" scale="0.001 0.001 0.001"/>
