Commit message: urdf tested with sensors
Signed-off-by: adrianco <adrian.cobo.mh@gmail.com>

File: description/lidar.xacro (robot description, xacro)
@@ -9,7 +9,7 @@
             <xacro:insert_block name="origin" />
             <parent link="${parent}"/>
-            <child link="rs_lidar" />
+            <child link="rslidar" />
         </joint>
-        <link name="rs_lidar">
+        <link name="rslidar">
             <visual name="">
                 <origin xyz="0.0 0.0 0.0" rpy="0.0 0.0 0.0"/>
