Commit message: urdf finished
Signed-off-by: adrianco <adrian.cobo.mh@gmail.com>

File: description/soporte.xacro (robot description, xacro)
@@ -9,12 +9,16 @@
     <xacro:include filename="jetson.xacro" />
     <xacro:include filename="$(find realsense2_description)/urdf/_d435.urdf.xacro" />
+    <xacro:include filename="box.xacro" />
     <xacro:lidar parent="lidar_chassis">
         <origin xyz="0.0 0.0 0.0575" rpy="0 0 0"/>
     </xacro:lidar>
     <xacro:jetson parent="base_footprint">
-        <origin xyz="0.0 0.0 -0.0365" rpy="0 0 0"/>
+        <origin xyz="0.065 0.0 -0.0365" rpy="0 0 0"/>
     </xacro:jetson>
     <xacro:sensor_d435 parent="camera_attachment_link" use_nominal_extrinsics="$(arg use_nominal_extrinsics)" add_plug="$(arg add_plug)" use_mesh="$(arg use_mesh)">
-        <origin xyz="0.01 0 -0.01" rpy="0 0 0"/>
+        <origin xyz="0.075 0 -0.01" rpy="0 0 0"/>
     </xacro:sensor_d435>
+    <xacro:box parent="base_footprint">
+        <origin xyz="0.0 0 -0.0" rpy="0 0 0"/>
+    </xacro:box>
 </robot>

File: description/soporte_core.xacro (robot description, xacro)
@@ -23,5 +23,5 @@
             <origin xyz="0.0 0.0 0.0" rpy="0.0 0.0 0.0"/>
             <geometry>
-                <mesh filename="package://perception_system/meshes/base.dae" scale="0.001 0.001 0.001"/>
+                <mesh filename="package://perception_system/meshes/base.dae"/>
             </geometry>
             <material name="white"/>
@@ -30,5 +30,5 @@
             <origin xyz="0 0.0 -0.005" rpy="0.0 0.0 0.0"/>
             <geometry>
-                <mesh filename="package://perception_system/meshes/base.dae" scale="0.001 0.001 0.001"/>
+                <mesh filename="package://perception_system/meshes/base.dae"/>
             </geometry>
         </collision>
@@ -45,5 +45,5 @@
     <link name="camera_attachment_link"></link>
     <joint name="lidar_chassis_joint" type="fixed">
-        <origin xyz="0.0 0.0 0.03" rpy="0.0 0.0 0.0"/>
+        <origin xyz="0.065 0.0 0.055" rpy="0.0 0.0 0.0"/>
         <parent link="base_footprint"/>
         <child link="lidar_chassis"/>
@@ -53,12 +53,12 @@
             <origin xyz="0.0 0.0 -0.03" rpy="0.0 0.0 0.0"/>
             <geometry>
-                <mesh filename="package://perception_system/meshes/soporte_lidar.dae" scale="0.001 0.001 0.001"/>
+                <mesh filename="package://perception_system/meshes/lidar_base.dae"/>
             </geometry>
             <material name="white"/>
         </visual>
         <collision>
-            <origin xyz="0 0.0 0.0" rpy="0.0 0.0 0.0"/>
+            <origin xyz="0 0.0 -0.03" rpy="0.0 0.0 0.0"/>
             <geometry>
-                <mesh filename="package://perception_system/meshes/soporte_lidar.dae" scale="0.001 0.001 0.001"/>
+                <mesh filename="package://perception_system/meshes/lidar_base.dae"/>
             </geometry>
         </collision>
